Commit message: newest branch

File: 41068_ws/src/41068_ignition_bringup/urdf/husky.gazebo.xacro (robot description, xacro)
@@ -140,5 +140,5 @@
     <sensor name="rgbd_camera" type="rgbd_camera">
       <camera>
-        <horizontal_fov>2.0944</horizontal_fov>
+        <horizontal_fov>1.5708</horizontal_fov>
         <image>
           <width>720</width>
@@ -164,5 +164,5 @@
       </camera>
       <always_on>1</always_on>
-      <update_rate>3</update_rate> <!--10-->
+      <update_rate>$(arg camera_update_rate)</update_rate>
       <visualize>$(arg camera_visual)</visualize>
       <topic>/model/husky/camera</topic>

File: 41068_ws/src/41068_ignition_bringup/urdf/husky.urdf.xacro (robot description, xacro)
@@ -1,4 +1,5 @@
 <?xml version="1.0" ?>
 <robot name="husky" xmlns:xacro="http://ros.org/wiki/xacro">
+  <xacro:arg name="camera_update_rate" default="30"/>
   <xacro:include filename="$(find 41068_ignition_bringup)/urdf/common_properties.urdf.xacro"/>
   <xacro:include filename="$(find 41068_ignition_bringup)/urdf/husky.gazebo.xacro"/>
@@ -121,5 +122,5 @@
   </link>
   <joint name="camera_joint" type="fixed">
-    <origin xyz="0.45 0.0 0.25" rpy="0 0 0"/> <!-- 0.5 0.0 0.9 -->
+    <origin xyz="0.45 0.0 0.20" rpy="0 -1.5708 0"/> <!-- Tilted to view trail -->
     <parent link="base_link"/>
     <child link="camera_link"/>
